File: kicad/pico-msxcart.kicad_sch (KiCad schematic)
At the start: 24 parts, among them J1 MSX-CONNECTOR, Q1 2N3904, U1 RaspberryPi_Pico, U10 AMS1117-3.3

Commit message: PCB Revision v0.1.0
Parts:
- added J2: ~, pico-msxcart:USB-A, symbol pico-msxcart:USB-A
Connections:
- net GND: now also J2.04 (GND)
- net VCC_4V7: now also J2.01 (VCC)
- new net: J2.S1 (SHIELD), J2.S2 (SHIELD)
- no-connect marks 5 -> 8
Changed lines of the file:
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@@
 	)
 	(no_connect
+		(at 247.65 154.94)
+	)
+	(no_connect
 		(at 259.08 91.44)
 	)
@@
 	)
 	(no_connect
+		(at 247.65 147.32)
+	)
+	(no_connect
 		(at 134.62 154.94)
 	)
@@
 	)
 	(no_connect
+		(at 247.65 144.78)
+	)
+	(no_connect
 		(at 149.86 157.48)
 	)
@@
 		)
 	)
+	(global_label "GND"
+		(shape input)
+		(at 247.65 149.86 180)
+		(fields_autoplaced yes)
+		(effects
+			(font
+				(size 1.27 1.27)
+			)
+			(justify right)
+		)
+		(property "Intersheetrefs" "${INTERSHEET_REFS}"
+			(at 240.7943 149.86 0)
+			(effects
+				(font
+					(size 1.27 1.27)
+				)
+				(justify right)
+				(hide yes)
+			)
+		)
+	)
 	(global_label "A5"
 		(shape output)
@@
 		)
 	)
+	(global_label "VCC_4V7"
+		(shape input)
+		(at 247.65 142.24 180)
+		(fields_autoplaced yes)
+		(effects
+			(font
+				(size 1.27 1.27)
+			)
+			(justify right)
+		)
+		(property "Intersheetrefs" "${INTERSHEET_REFS}"
+			(at 236.561 142.24 0)
+			(effects
+				(font
+					(size 1.27 1.27)
+				)
+				(justify right)
+				(hide yes)
+			)
+		)
+	)
 	(global_label "D3"
 		(shape bidirectional)
@@
 					(unit 1)
 				)
+			)
+		)
+	)
+	(symbol
+		(lib_id "pico-msxcart:USB-A")
+		(at 257.81 147.32 0)
+		(unit 1)
+		(exclude_from_sim no)
+		(in_bom yes)
+		(on_board yes)
+		(dnp no)
+		(fields_autoplaced yes)
+		(property "Reference" "J2"
+			(at 264.16 147.9549 0)
+			(effects
+				(font
+					(size 1.27 1.27)
+				)
+				(justify left)
+			)
+		)
+		(property "Value" "~"
+			(at 264.16 149.86 0)
+			(effects
+				(font
+					(size 1.27 1.27)
+				)
+				(justify left)
+			)
+		)
+		(property "Footprint" "pico-msxcart:USB-A"
+			(at 257.81 138.43 0)
+			(effects
+				(font
+					(size 1.27 1.27)
+				)
+				(hide yes)
+			)
+		)
+		(property "Datasheet" ""
+			(at 257.81 138.43 0)
+			(effects
+				(font
+					(size 1.27 1.27)
+				)
+				(hide yes)
+			)
+		)
+		(property "Description" ""
+			(at 257.81 138.43 0)
+			(effects
+				(font
+					(size 1.27 1.27)
+				)
+				(hide yes)
+			)
+		)
+		(pin "S2"
+		)
+		(pin "S1"
+		)
+		(pin "03"
+		)
+		(pin "04"
+		)
+		(pin "01"
+		)
+		(pin "02"
+		)
+		(instances
+			(project "pico-msxcart"
+				(path "/c6ea766e-7213-4fff-afb7-62b69cefee35"
+					(reference "J2")
+					(unit 1)
+				)

Commit message: Switched to Patola Board
Parts:
- added R3, R4: 2k2, pico-msxcart:R0603, symbol pico-msxcart:SMD_RESISTOR
- added TP11: ~, pico-msxcart:TEST_PROBE, symbol pico-msxcart:TEST_PROBE
- added U7: ~, pico-msxcart:SOP-14, symbol pico-msxcart:SN74LS00
- D1: footprint pico-msxcart:SCHOTKKY -> pico-msxcart:SCHOTKKY_THT
- J1: footprint pico-msxcart:MSX-CONNECTOR2 -> pico-msxcart:MSXCART
Connections:
- net D0_3V3 is gone; now on net MP0_3V3: U1.1 (GPIO0), U4.18 (B0)
- net D1_3V3 is gone; now on net MP1_3V3: U1.2 (GPIO1), U4.17 (B1)
- net D2_3V3 is gone; now on net MP2_3V3: U1.4 (GPIO2), U4.16 (B2)
- net D3_3V3 is gone; now on net MP3_3V3: U1.5 (GPIO3), U4.15 (B3)
- net D4_3V3 is gone; now on net MP4_3V3: U1.6 (GPIO4), U4.14 (B4)
- net D5_3V3 is gone; now on net MP5_3V3: U1.7 (GPIO5), U4.13 (B5)
- net D6_3V3 is gone; now on net MP6_3V3: U1.9 (GPIO6), U4.12 (B6)
- net D7_3V3 is gone; now on net MP7_3V3: U1.10 (GPIO7), U4.11 (B7)
- net BUSDIR3V3: now also U1.24 (GPIO18); no longer U1.26 (GPIO20)
- net CS12: now also U5.6 (A4); no longer U5.8 (A6)
- net DATADIR: now also U1.22 (GPIO17); no longer U1.25 (GPIO19)
- net GND: now also TP7.1 (PROBE), U5.9 (A7), U7.10 (3B), U7.12 (4A), U7.13 (4B), U7.4 (2A), U7.5 (2B), U7.7 (GND), U7.9 (3A); no longer TP7. (PROBE), U4.19 (~{OE})
- net INT3V3: now also U1.25 (GPIO19); no longer U1.27 (GPIO21)
- net M1: now also U5.8 (A6); no longer U5.9 (A7)
- net MP0_3V3: no longer U1.11 (GPIO8), U3.18 (B0), U5.18 (B0)
- net MP1_3V3: no longer U1.12 (GPIO9), U3.17 (B1), U5.17 (B1)
- net MP2_3V3: no longer U1.14 (GPIO10), U3.16 (B2), U5.16 (B2)
- net MP3_3V3: no longer U1.15 (GPIO11), U3.15 (B3), U5.15 (B3)
- net MP4_3V3: no longer U1.16 (GPIO12), U3.14 (B4), U5.14 (B4)
- net MP5_3V3: no longer U1.17 (GPIO13), U3.13 (B5), U5.13 (B5)
- net MP6_3V3: no longer U1.19 (GPIO14), U3.12 (B6), U5.12 (B6)
- net MP7_3V3: no longer U1.20 (GPIO15), U3.11 (B7), U5.11 (B7)
- net MSEL0_3V3: now also U3.19 (~{OE}), U7.1 (1A), U7.2 (1B)
- net MSEL1_3V3: now also U4.19 (~{OE}), U5.19 (~{OE}), U7.3 (1Y); no longer U1.22 (GPIO17), U3.19 (~{OE})
- net RD_3V3: now also U1.26 (GPIO20); no longer U1.29 (GPIO22)
- net RESET: now also U6.9 (A7); no longer U5.6 (A4)
- net VCC: now also TP6.1 (PROBE); no longer TP6. (PROBE)
- net VCC_3V3: now also TP5.1 (PROBE), R3.2, R4.2, U7.14 (VCC); no longer TP5. (PROBE)
- net VCC_4V7: now also TP4.1 (PROBE); no longer TP4. (PROBE)
- net WR_3V3: now also U1.27 (GPIO21); no longer U1.31 (GPIO26_ADC0)
- net at J1.48 (+12): now also TP2.1 (PROBE); no longer TP2. (PROBE)
- net at J1.49 (SOUNDIN): now also TP1.1 (PROBE); no longer TP1. (PROBE)
- net at J1.16 (RSV@2): now also TP9.1 (PROBE); no longer TP9. (PROBE)
- net at J1.5 (RSV@1): now also TP8.1 (PROBE); no longer TP8. (PROBE)
- net at J1.50 (-12): now also TP3.1 (PROBE); no longer TP3. (PROBE)
- net RUN: now reaches U1.30 (RUN)
- net RUN: now also TP10.1 (PROBE), R3.1; no longer TP10. (PROBE)
- net 3V3_EN: now reaches U1.37 (3V3_EN)
- net 3V3_EN: now also R4.1, TP11.1 (PROBE)
- net RESET_3V3: now reaches U6.11 (B7)
- net RESET_3V3: now also U1.31 (GPIO26_ADC0)
- removed net MSEL2_3V3: U1.24 (GPIO18), U5.19 (~{OE})
- new net MP10_3V3: U1.14 (GPIO10), U3.16 (B2), U5.16 (B2)
- new net MP11_3V3: U1.15 (GPIO11), U3.15 (B3), U5.15 (B3)
- new net MP12_3V3: U1.16 (GPIO12), U3.14 (B4), U5.14 (B4)
- new net MP13_3V3: U1.17 (GPIO13), U3.13 (B5), U5.13 (B5)
- new net MP14_3V3: U1.19 (GPIO14), U3.12 (B6), U5.12 (B6)
- new net MP15_3V3: U1.20 (GPIO15), U3.11 (B7), U5.11 (B7)
- new net MP8_3V3: U1.11 (GPIO8), U3.18 (B0), U5.18 (B0)
- new net MP9_3V3: U1.12 (GPIO9), U3.17 (B1), U5.17 (B1)
- no-connect marks 8 -> 10
Other:
- company: (none) -> Chandler Klüser
- title: (none) -> PicoMSX
- moved on the sheet: Q1, R1, R2, TP10, U2, U3, U4, U5, U6
